Commit message: 주행 테스트

File: src/vic_pinky/vicpinky_description/urdf/robot_core.xacro (robot description, xacro)
@@ -142,4 +142,9 @@
         </xacro:inertial_cylinder>
     </link>
+    <!-- <joint name="${prefix}left_caster_joint" type="fixed">
+        <parent link="${prefix}base_link"/>
+        <child link="${prefix}left_caster"/>
+        <origin xyz="${-chassis_length/2-0.1} ${chassis_width/2-0.1} ${-caster_wheel_radius}" rpy="0 0 0"/>
+    </joint> -->
     <joint name="${prefix}left_caster_joint" type="fixed">
         <parent link="${prefix}base_link"/>
@@ -165,4 +170,9 @@
         </xacro:inertial_sphere>
     </link>
+    <!-- <joint name="${prefix}right_caster_joint" type="fixed">
+        <parent link="${prefix}base_link"/>
+        <child link="${prefix}right_caster"/>
+        <origin xyz="${-chassis_length/2-0.1} ${-chassis_width/2+0.1} ${-caster_wheel_radius}" rpy="0 0 0"/>
+    </joint> -->
     <joint name="${prefix}right_caster_joint" type="fixed">
         <parent link="${prefix}base_link"/>
@@ -233,5 +243,5 @@
         <parent link="${prefix}lidar_mount"/>
         <child link="${prefix}laser_link"/>
-        <origin xyz="0.0 0 0.03" rpy="0 0 ${pi}"/>
+        <origin xyz="0.0 0 0.03" rpy="0 0 0"/>
     </joint>
 </robot>
